Commit message: Fixing names.

File: simplebot_description/urdf/simplebot.urdf.xacro (robot description, xacro)
@@ -205,21 +205,21 @@
     <origin xyz="-0.014 -0.05 0.222" rpy="0 0 0"/>
   </joint>
-  <link name="lidar3d_plate_link">
-    <visual>
-      <origin xyz="0 0 0" rpy="0 0 0"/>
-      <geometry>
-        <box size="0.14 0.14 0.005"/>
-      </geometry>
-      <material name="grey"/>
-    </visual>
-  </link>
-  <joint name="platform_support_leg1_link_to_lidar3d_plate_link" type="fixed">
-    <parent link="platform_support_leg1_link"/>
-    <child link="lidar3d_plate_link"/>
-    <origin xyz="0.05 -0.05 0" rpy="0 0 0"/>
-  </joint>
-  <xacro:VLP-16 name="lidar3d" parent="lidar3d_plate_link" topic="/lidar3d/points">
-    <origin xyz="0 0 0" rpy="0 0 0" />
-  </xacro:VLP-16>
+<!--  <link name="lidar3d_plate_link">-->
+<!--    <visual>-->
+<!--      <origin xyz="0 0 0" rpy="0 0 0"/>-->
+<!--      <geometry>-->
+<!--        <box size="0.14 0.14 0.005"/>-->
+<!--      </geometry>-->
+<!--      <material name="grey"/>-->
+<!--    </visual>-->
+<!--  </link>-->
+<!--  <joint name="platform_support_leg1_link_to_lidar3d_plate_link" type="fixed">-->
+<!--    <parent link="platform_support_leg1_link"/>-->
+<!--    <child link="lidar3d_plate_link"/>-->
+<!--    <origin xyz="0.05 -0.05 0" rpy="0 0 0"/>-->
+<!--  </joint>-->
+<!--  <xacro:VLP-16 name="lidar3d" parent="lidar3d_plate_link" topic="/lidar3d/points">-->
+<!--    <origin xyz="0 0 0" rpy="0 0 0" />-->
+<!--  </xacro:VLP-16>-->
   <link name="front_left_camera_support_link">
   </link>
@@ -232,23 +232,50 @@
     <origin xyz="0.02 0.07 0.015" rpy="0 0.0 0" />
   </xacro:sensor_astra>
-  <link name="front_right_camera_support_link">
-  </link>
-  <joint name="platform_support_leg4_link_to_front_right_camera_support_link" type="fixed">
-    <origin xyz="0.02 0 -0.05" rpy="0.01 -0.35 -0.22"/>
-    <parent link="platform_support_leg4_link"/>
-    <child link="front_right_camera_support_link"/>
-  </joint>
-  <xacro:sensor_astra prefix="front_right_camera" parent="front_right_camera_support_link">
-    <origin xyz="0.02 0.07 0.015" rpy="0 0.0 0" />
-  </xacro:sensor_astra>
-  <link name="back_camera_support_link">
-  </link>
-  <joint name="platform_support_leg1_link_to_back_camera_support_link" type="fixed">
-    <origin xyz="-0.02 -0.05 -0.10" rpy="0.01 -0.35 3.14"/>
-    <parent link="platform_support_leg1_link"/>
-    <child link="back_camera_support_link"/>
-  </joint>
-  <xacro:sensor_astra prefix="back_camera" parent="back_camera_support_link">
-    <origin xyz="0.02 0.07 0.015" rpy="0 0.0 0" />
-  </xacro:sensor_astra>
+<!--  <link name="front_right_camera_support_link">-->
+<!--  </link>-->
+<!--  <joint name="platform_support_leg4_link_to_front_right_camera_support_link" type="fixed">-->
+<!--    <origin xyz="0.02 0 -0.05" rpy="0.01 -0.35 -0.22"/>-->
+<!--    <parent link="platform_support_leg4_link"/>-->
+<!--    <child link="front_right_camera_support_link"/>-->
+<!--  </joint>-->
+<!--  <xacro:sensor_astra prefix="front_right_camera" parent="front_right_camera_support_link">-->
+<!--    <origin xyz="0.02 0.07 0.015" rpy="0 0.0 0" />-->
+<!--  </xacro:sensor_astra>-->
+<!--  <link name="back_camera_support_link">-->
+<!--  </link>-->
+<!--  <joint name="platform_support_leg1_link_to_back_camera_support_link" type="fixed">-->
+<!--    <origin xyz="-0.02 -0.05 -0.10" rpy="0.01 -0.35 3.14"/>-->
+<!--    <parent link="platform_support_leg1_link"/>-->
+<!--    <child link="back_camera_support_link"/>-->
+<!--  </joint>-->
+<!--  <xacro:sensor_astra prefix="back_camera" parent="back_camera_support_link">-->
+<!--    <origin xyz="0.02 0.07 0.015" rpy="0 0.0 0" />-->
+<!--  </xacro:sensor_astra>-->
+ <joint name="scan_joint" type="fixed">
+    <parent link="base_link"/>
+    <child link="base_scan"/>
+    <origin xyz="-0.064 0 0.122" rpy="0 0 0"/>
+  </joint>
+  <link name="base_scan">
+    <visual>
+      <origin xyz="0 0 0.0" rpy="0 0 0"/>
+      <geometry>
+        <mesh filename="package://turtlebot3_description/meshes/sensors/lds.stl" scale="0.001 0.001 0.001"/>
+      </geometry>
+      <material name="dark"/>
+    </visual>
+    <collision>
+      <origin xyz="0.015 0 -0.0065" rpy="0 0 0"/>
+      <geometry>
+        <cylinder length="0.0315" radius="0.055"/>
+      </geometry>
+    </collision>
+    <inertial>
+      <mass value="0.114" />
+      <origin xyz="0 0 0" />
+      <inertia ixx="0.001" ixy="0.0" ixz="0.0"
+               iyy="0.001" iyz="0.0"
+               izz="0.001" />
+    </inertial>
+  </link>
 </robot>
