Commit message: Adding two 2d lidars

File: simplebot_description/urdf/simplebot.gazebo.macro.xacro (robot description, xacro)
@@ -99,23 +99,23 @@
     </plugin>
   </gazebo>
-  <gazebo reference="base_scan">
+  <gazebo reference="left_base_scan">
     <material>Gazebo/FlatBlack</material>
-    <sensor type="ray" name="lds_lfcd_sensor">
+    <sensor type="ray" name="lds_lfcd_sensor_left">
       <pose>0 0 0 0 0 0</pose>
-      <visualize>${laser_visual}</visualize>
-<!--      <visualize>true</visualize>-->
+<!--      <visualize>${laser_visual}</visualize>-->
+      <visualize>true</visualize>
       <update_rate>5</update_rate>
       <ray>
         <scan>
           <horizontal>
-            <samples>360</samples>
+            <samples>180</samples>
             <resolution>1</resolution>
-            <min_angle>0.0</min_angle>
-            <max_angle>6.28319</max_angle>
+            <min_angle>-1.57</min_angle>
+            <max_angle>1.57</max_angle>
           </horizontal>
         </scan>
         <range>
           <min>0.120</min>
-          <max>3.5</max>
+          <max>5.5</max>
           <resolution>0.015</resolution>
         </range>
@@ -127,6 +127,39 @@
       </ray>
       <plugin name="gazebo_ros_lds_lfcd_controller" filename="libgazebo_ros_laser.so">
-        <topicName>scan</topicName>
-        <frameName>base_scan</frameName>
+        <topicName>left_scan</topicName>
+        <frameName>left_base_scan</frameName>
+      </plugin>
+    </sensor>
+  </gazebo>
+    <gazebo reference="right_base_scan">
+    <material>Gazebo/FlatBlack</material>
+    <sensor type="ray" name="lds_lfcd_sensor_right">
+      <pose>0 0 0 0 0 0</pose>
+<!--      <visualize>${laser_visual}</visualize>-->
+      <visualize>true</visualize>
+      <update_rate>5</update_rate>
+      <ray>
+        <scan>
+          <horizontal>
+            <samples>180</samples>
+            <resolution>1</resolution>
+            <min_angle>-1.57</min_angle>
+            <max_angle>1.57</max_angle>
+          </horizontal>
+        </scan>
+        <range>
+          <min>0.120</min>
+          <max>5.5</max>
+          <resolution>0.015</resolution>
+        </range>
+        <noise>
+          <type>gaussian</type>
+          <mean>0.0</mean>
+          <stddev>0.01</stddev>
+        </noise>
+      </ray>
+      <plugin name="gazebo_ros_lds_lfcd_controller" filename="libgazebo_ros_laser.so">
+        <topicName>right_scan</topicName>
+        <frameName>right_base_scan</frameName>
       </plugin>
     </sensor>

File: simplebot_description/urdf/simplebot.urdf.xacro (robot description, xacro)
@@ -252,10 +252,11 @@
 <!--    <origin xyz="0.02 0.07 0.015" rpy="0 0.0 0" />-->
 <!--  </xacro:sensor_astra>-->
- <joint name="scan_joint" type="fixed">
-    <parent link="base_link"/>
-    <child link="base_scan"/>
-    <origin xyz="-0.064 0 0.122" rpy="0 0 0"/>
-  </joint>
-  <link name="base_scan">
+ <joint name="left_scan_joint" type="fixed">
+    <parent link="base_link"/>
+    <child link="left_base_scan"/>
+<!--    <origin xyz="-0.064 0 0.122" rpy="0 0 0"/>-->
+   <origin xyz="0.037 0.1 0.122" rpy="0 0 0.78"/>
+  </joint>
+  <link name="left_base_scan">
     <visual>
       <origin xyz="0 0 0.0" rpy="0 0 0"/>
@@ -272,5 +273,5 @@
     </collision>
     <inertial>
-      <mass value="0.114" />
+      <mass value="0.0" />
       <origin xyz="0 0 0" />
       <inertia ixx="0.001" ixy="0.0" ixz="0.0"
@@ -279,3 +280,31 @@
     </inertial>
   </link>
+   <joint name="right_scan_joint" type="fixed">
+    <parent link="base_link"/>
+    <child link="right_base_scan"/>
+<!--    <origin xyz="-0.064 0 0.122" rpy="0 0 0"/>-->
+   <origin xyz="0.037 -0.1 0.122" rpy="0 0 -0.78"/>
+  </joint>
+  <link name="right_base_scan">
+    <visual>
+      <origin xyz="0 0 0.0" rpy="0 0 0"/>
+      <geometry>
+        <mesh filename="package://turtlebot3_description/meshes/sensors/lds.stl" scale="0.001 0.001 0.001"/>
+      </geometry>
+      <material name="dark"/>
+    </visual>
+    <collision>
+      <origin xyz="0.015 0 -0.0065" rpy="0 0 0"/>
+      <geometry>
+        <cylinder length="0.0315" radius="0.055"/>
+      </geometry>
+    </collision>
+    <inertial>
+      <mass value="0.0" />
+      <origin xyz="0 0 0" />
+      <inertia ixx="0.001" ixy="0.0" ixz="0.0"
+               iyy="0.001" iyz="0.0"
+               izz="0.001" />
+    </inertial>
+  </link>
 </robot>
