Commit message: #61 working cmf estimation

File: simplebot_calibration/urdf/initial_estimate.urdf.xacro (robot description, xacro)
@@ -1,30 +1,230 @@
 <?xml version="1.0" ?>
-<robot name="simplebot" xmlns:xacro="http://ros.org/wiki/xacro">
-  <!--  Xacro description of turtlebot robot waffle pi used to play team hunt.-->
-  <!--  Miguel Riem Oliveira-->
-  <!--  PARI, November 2020-->
-  <!--Args are local, properties are global, so we copy the values of the arguments to the properties-->
-  <xacro:arg name="name" default="simplebot" />
-  <xacro:arg name="color" default="Orange" /> <!-- e.g. Red, Orange. Must exist in Gazebo/Colors and be defined in properties.xacro.-->
-  <!--Properties are global so they can be viewed from inside the included xacros-->
-  <!--  args are used with $(arg arg_name), properties are used as ${property_name}-->
-  <xacro:property name="name" value="$(arg name)"/>
-  <xacro:property name="color" value="$(arg color)"/>
-  <!-- Include other files-->
-  <xacro:include filename="$(find simplebot_description)/urdf/properties.xacro"/>
-  <xacro:include filename="$(find simplebot_description)/urdf/VLP-16.urdf.xacro"/>
-  <xacro:include filename="$(find simplebot_description)/urdf/astra.urdf.xacro" />
-  <xacro:include filename="$(find simplebot_description)/urdf/simplebot.gazebo.macro.xacro"/>
-  <xacro:gazebo_macro color="$(arg color)" laser_visual="false" camera_visual="false" imu_visual="true"/>
-  <!-- Links and joints-->
+<robot name="simplebot" version="1.0">
+  <material name="black">
+    <color rgba="0.0 0.0 0.0 1.0"/>
+  </material>
+  <material name="dark">
+    <color rgba="0.3 0.3 0.3 1.0"/>
+  </material>
+  <material name="light_black">
+    <color rgba="0.4 0.4 0.4 1.0"/>
+  </material>
+  <material name="blue">
+    <color rgba="0.0 0.0 0.8 1.0"/>
+  </material>
+  <material name="green">
+    <color rgba="0.0 0.8 0.0 1.0"/>
+  </material>
+  <material name="grey">
+    <color rgba="0.5 0.5 0.5 1.0"/>
+  </material>
+  <material name="orange">
+    <color rgba="1.0 0.4235294117647059 0.0392156862745098 1.0"/>
+  </material>
+  <material name="brown">
+    <color rgba="0.8705882352941177 0.8117647058823529 0.7647058823529411 1.0"/>
+  </material>
+  <material name="red">
+    <color rgba="0.8 0.0 0.0 1.0"/>
+  </material>
+  <material name="white">
+    <color rgba="1.0 1.0 1.0 1.0"/>
+  </material>
+  <material name="Yellow">
+    <color rgba="1.0 1.0 0.0 1.0"/>
+  </material>
+  <material name="Orange">
+    <color rgba="1.0 0.4 0.0 1.0"/>
+  </material>
+  <material name="Gray">
+    <color rgba="1.0 0.4 0.0 1.0"/>
+  </material>
+  <gazebo reference="base_link">
+    <material>Gazebo/Orange</material>
+  </gazebo>
+  <gazebo reference="base_link">
+    <sensor name="base_link" type="contact">
+      <update_rate>1000.0</update_rate>
+      <always_on>true</always_on>
+      <contact>
+        <collision>base_footprint_fixed_joint_lump__base_link_collision_collision</collision>
+      </contact>
+      <plugin filename="libgazebo_ros_bumper.so" name="base_link_contact_sensor_plugin">
+        <bumperTopicName>contact</bumperTopicName>
+        <frameName>world</frameName>
+      </plugin>
+    </sensor>
+  </gazebo>
+  <gazebo reference="wheel_left_link">
+    <mu1>0.1</mu1>
+    <mu2>0.1</mu2>
+    <kp>500000.0</kp>
+    <kd>10.0</kd>
+    <minDepth>0.001</minDepth>
+    <maxVel>0.1</maxVel>
+    <fdir1>1 0 0</fdir1>
+    <material>Gazebo/Orange</material>
+  </gazebo>
+  <gazebo reference="wheel_right_link">
+    <mu1>0.1</mu1>
+    <mu2>0.1</mu2>
+    <kp>500000.0</kp>
+    <kd>10.0</kd>
+    <minDepth>0.001</minDepth>
+    <maxVel>0.01</maxVel>
+    <fdir1>1 0 0</fdir1>
+    <material>Gazebo/Orange</material>
+  </gazebo>
+  <gazebo reference="caster_back_right_link">
+    <mu1>0.1</mu1>
+    <mu2>0.1</mu2>
+    <kp>1000000.0</kp>
+    <kd>100.0</kd>
+    <minDepth>0.001</minDepth>
+    <maxVel>1.0</maxVel>
+    <material>Gazebo/FlatBlack</material>
+  </gazebo>
+  <gazebo reference="caster_back_left_link">
+    <mu1>0.1</mu1>
+    <mu2>0.1</mu2>
+    <kp>1000000.0</kp>
+    <kd>100.0</kd>
+    <minDepth>0.001</minDepth>
+    <maxVel>1.0</maxVel>
+    <material>Gazebo/FlatBlack</material>
+  </gazebo>
+  <gazebo reference="imu_link">
+    <sensor name="imu" type="imu">
+      <always_on>true</always_on>
+      <visualize>True</visualize>
+    </sensor>
+    <material>Gazebo/Grey</material>
+  </gazebo>
+  <gazebo>
+    <plugin filename="libgazebo_ros_diff_drive.so" name="turtlebot3_waffle_pi_controller">
+      <commandTopic>cmd_vel</commandTopic>
+      <odometryTopic>odom</odometryTopic>
+      <odometryFrame>world</odometryFrame>
+      <odometrySource>world</odometrySource>
+      <publishOdomTF>true</publishOdomTF>
+      <robotBaseFrame>base_footprint</robotBaseFrame>
+      <publishWheelTF>false</publishWheelTF>
+      <publishTf>true</publishTf>
+      <publishWheelJointState>true</publishWheelJointState>
+      <legacyMode>false</legacyMode>
+      <updateRate>30</updateRate>
+      <leftJoint>wheel_left_joint</leftJoint>
+      <rightJoint>wheel_right_joint</rightJoint>
+      <wheelSeparation>0.287</wheelSeparation>
+      <wheelDiameter>0.066</wheelDiameter>
+      <wheelAcceleration>1</wheelAcceleration>
+      <wheelTorque>10</wheelTorque>
+      <rosDebugLevel>na</rosDebugLevel>
+    </plugin>
+  </gazebo>
+  <gazebo>
+    <plugin filename="libgazebo_ros_imu.so" name="imu_plugin">
+      <alwaysOn>true</alwaysOn>
+      <bodyName>imu_link</bodyName>
+      <frameName>imu_link</frameName>
+      <topicName>imu</topicName>
+      <serviceName>imu_service</serviceName>
+      <gaussianNoise>0.0</gaussianNoise>
+      <updateRate>200</updateRate>
+      <imu>
+        <noise>
+          <type>gaussian</type>
+          <rate>
+            <mean>0.0</mean>
+            <stddev>2e-4</stddev>
+            <bias_mean>0.0000075</bias_mean>
+            <bias_stddev>0.0000008</bias_stddev>
+          </rate>
+          <accel>
+            <mean>0.0</mean>
+            <stddev>1.7e-2</stddev>
+            <bias_mean>0.1</bias_mean>
+            <bias_stddev>0.001</bias_stddev>
+          </accel>
+        </noise>
+      </imu>
+    </plugin>
+  </gazebo>
+  <gazebo reference="left_base_scan">
+    <material>Gazebo/FlatBlack</material>
+    <sensor name="lds_lfcd_sensor_left" type="ray">
+      <pose>0 0 0 0 0 0</pose>
+      <update_rate>5</update_rate>
+      <ray>
+        <scan>
+          <horizontal>
+            <samples>180</samples>
+            <resolution>1</resolution>
+            <min_angle>-1.57</min_angle>
+            <max_angle>1.57</max_angle>
+          </horizontal>
+        </scan>
+        <range>
+          <min>0.120</min>
+          <max>5.5</max>
+          <resolution>0.015</resolution>
+        </range>
+        <noise>
+          <type>gaussian</type>
+          <mean>0.0</mean>
+          <stddev>0.01</stddev>
+        </noise>
+      </ray>
+      <plugin filename="libgazebo_ros_laser.so" name="gazebo_ros_lds_lfcd_controller">
+        <topicName>left_scan</topicName>
+        <frameName>left_base_scan</frameName>
+      </plugin>
+    </sensor>
+  </gazebo>
+  <gazebo reference="right_base_scan">
+    <material>Gazebo/FlatBlack</material>
+    <sensor name="lds_lfcd_sensor_right" type="ray">
+      <pose>0 0 0 0 0 0</pose>
+      <update_rate>5</update_rate>
+      <ray>
+        <scan>
+          <horizontal>
+            <samples>180</samples>
+            <resolution>1</resolution>
+            <min_angle>-1.57</min_angle>
+            <max_angle>1.57</max_angle>
+          </horizontal>
+        </scan>
+        <range>
+          <min>0.120</min>
+          <max>5.5</max>
+          <resolution>0.015</resolution>
+        </range>
+        <noise>
+          <type>gaussian</type>
+          <mean>0.0</mean>
+          <stddev>0.01</stddev>
+        </noise>
+      </ray>
+      <plugin filename="libgazebo_ros_laser.so" name="gazebo_ros_lds_lfcd_controller">
+        <topicName>right_scan</topicName>
+        <frameName>right_base_scan</frameName>
+      </plugin>
+    </sensor>
+  </gazebo>
   <link name="base_footprint"/>
   <joint name="base_joint" type="fixed">
+    <origin xyz="0.0 0.0 0.01" rpy="0.0 0.0 0.0"/>
     <parent link="base_footprint"/>
-    <child link="base_link" />
-    <origin xyz="0 0 0.010" rpy="0 0 0"/>
+    <child link="base_link"/>
   </joint>
   <link name="base_link">
-    <visual>
-      <origin xyz="-0.064 0 0.0" rpy="0 0 0"/>
+    <inertial>
+      <origin xyz="0.0 0.0 0.0" rpy="0.0 0.0 0.0"/>
+      <mass value="1.3729096"/>
+      <inertia ixx="0.0087002718" ixy="-4.7576583e-05" ixz="0.00011160499" iyy="0.0086195418" iyz="-3.5422299e-06" izz="0.014612727"/>
+    </inertial>
+    <visual>
+      <origin xyz="-0.064 0.0 0.0" rpy="0.0 0.0 0.0"/>
       <geometry>
         <mesh filename="package://turtlebot3_description/meshes/bases/waffle_pi_base.stl" scale="0.001 0.001 0.001"/>
@@ -33,27 +233,24 @@
     </visual>
     <collision name="base_link_collision">
-      <origin xyz="-0.064 0 0.047" rpy="0 0 0"/>
-      <geometry>
-        <!--        <box size="0.266 0.266 0.094"/>-->
+      <origin xyz="-0.064 0.0 0.047" rpy="0.0 0.0 0.0"/>
+      <geometry>
         <box size="0.3 0.3 0.094"/>
       </geometry>
     </collision>
-    <inertial>
-      <origin xyz="0 0 0" rpy="0 0 0"/>
-      <mass value="1.3729096e+00"/>
-      <inertia ixx="8.7002718e-03" ixy="-4.7576583e-05" ixz="1.1160499e-04"
-               iyy="8.6195418e-03" iyz="-3.5422299e-06"
-               izz="1.4612727e-02" />
-    </inertial>
   </link>
   <joint name="wheel_left_joint" type="continuous">
+    <origin xyz="0.0 0.144 0.023" rpy="-1.57 0.0 0.0"/>
+    <axis xyz="0.0 0.0 1.0"/>
     <parent link="base_link"/>
     <child link="wheel_left_link"/>
-    <origin xyz="0.0 0.144 0.023" rpy="-1.57 0 0"/>
-    <axis xyz="0 0 1"/>
   </joint>
   <link name="wheel_left_link">
-    <visual>
-      <origin xyz="0 0 0" rpy="1.57 0 0"/>
+    <inertial>
+      <origin xyz="0.0 0.0 0.0" rpy="0 0 0"/>
+      <mass value="0.02849894"/>
+      <inertia ixx="1.117558e-05" ixy="-4.2369783e-11" ixz="-5.9381719e-09" iyy="1.1192413e-05" iyz="-1.4400107e-11" izz="2.0712558e-05"/>
+    </inertial>
+    <visual>
+      <origin xyz="0.0 0.0 0.0" rpy="1.57 0.0 0.0"/>
       <geometry>
         <mesh filename="package://turtlebot3_description/meshes/wheels/left_tire.stl" scale="0.001 0.001 0.001"/>
@@ -62,26 +259,24 @@
     </visual>
     <collision>
-      <origin xyz="0 0 0" rpy="0 0 0"/>
-      <geometry>
-        <cylinder length="0.018" radius="0.033"/>
-      </geometry>
-    </collision>
-    <inertial>
-      <origin xyz="0 0 0" />
-      <mass value="2.8498940e-02" />
-      <inertia ixx="1.1175580e-05" ixy="-4.2369783e-11" ixz="-5.9381719e-09"
-               iyy="1.1192413e-05" iyz="-1.4400107e-11"
-               izz="2.0712558e-05" />
-    </inertial>
+      <origin xyz="0.0 0.0 0.0" rpy="0.0 0.0 0.0"/>
+      <geometry>
+        <cylinder radius="0.033" length="0.018"/>
+      </geometry>
+    </collision>
   </link>
   <joint name="wheel_right_joint" type="continuous">
+    <origin xyz="0.0 -0.144 0.023" rpy="-1.57 0.0 0.0"/>
+    <axis xyz="0.0 0.0 1.0"/>
     <parent link="base_link"/>
     <child link="wheel_right_link"/>
-    <origin xyz="0.0 -0.144 0.023" rpy="-1.57 0 0"/>
-    <axis xyz="0 0 1"/>
   </joint>
   <link name="wheel_right_link">
-    <visual>
-      <origin xyz="0 0 0" rpy="1.57 0 0"/>
+    <inertial>
+      <origin xyz="0.0 0.0 0.0" rpy="0 0 0"/>
+      <mass value="0.02849894"/>
+      <inertia ixx="1.117558e-05" ixy="-4.2369783e-11" ixz="-5.9381719e-09" iyy="1.1192413e-05" iyz="-1.4400107e-11" izz="2.0712558e-05"/>
+    </inertial>
+    <visual>
+      <origin xyz="0.0 0.0 0.0" rpy="1.57 0.0 0.0"/>
       <geometry>
         <mesh filename="package://turtlebot3_description/meshes/wheels/right_tire.stl" scale="0.001 0.001 0.001"/>
@@ -90,68 +285,57 @@
     </visual>
     <collision>
-      <origin xyz="0 0 0" rpy="0 0 0"/>
-      <geometry>
-        <cylinder length="0.018" radius="0.033"/>
-      </geometry>
-    </collision>
-    <inertial>
-      <origin xyz="0 0 0" />
-      <mass value="2.8498940e-02" />
-      <inertia ixx="1.1175580e-05" ixy="-4.2369783e-11" ixz="-5.9381719e-09"
-               iyy="1.1192413e-05" iyz="-1.4400107e-11"
-               izz="2.0712558e-05" />
-    </inertial>
+      <origin xyz="0.0 0.0 0.0" rpy="0.0 0.0 0.0"/>
+      <geometry>
+        <cylinder radius="0.033" length="0.018"/>
+      </geometry>
+    </collision>
   </link>
   <joint name="caster_back_right_joint" type="fixed">
+    <origin xyz="-0.177 -0.064 -0.004" rpy="-1.57 0.0 0.0"/>
     <parent link="base_link"/>
     <child link="caster_back_right_link"/>
-    <origin xyz="-0.177 -0.064 -0.004" rpy="-1.57 0 0"/>
   </joint>
   <link name="caster_back_right_link">
-    <collision>
-      <origin xyz="0 0.001 0" rpy="0 0 0"/>
-      <geometry>
-        <box size="0.030 0.009 0.020"/>
-      </geometry>
-    </collision>
-    <inertial>
-      <origin xyz="0 0 0" />
-      <mass value="0.005" />
-      <inertia ixx="0.001" ixy="0.0" ixz="0.0"
-               iyy="0.001" iyz="0.0"
-               izz="0.001" />
-    </inertial>
+    <inertial>
+      <origin xyz="0.0 0.0 0.0" rpy="0 0 0"/>
+      <mass value="0.005"/>
+      <inertia ixx="0.001" ixy="0.0" ixz="0.0" iyy="0.001" iyz="0.0" izz="0.001"/>
+    </inertial>
+    <collision>
+      <origin xyz="0.0 0.001 0.0" rpy="0.0 0.0 0.0"/>
+      <geometry>
+        <box size="0.03 0.009 0.02"/>
+      </geometry>
+    </collision>
   </link>
   <joint name="caster_back_left_joint" type="fixed">
+    <origin xyz="-0.177 0.064 -0.004" rpy="-1.57 0.0 0.0"/>
     <parent link="base_link"/>
     <child link="caster_back_left_link"/>
-    <origin xyz="-0.177 0.064 -0.004" rpy="-1.57 0 0"/>
   </joint>
   <link name="caster_back_left_link">
-    <collision>
-      <origin xyz="0 0.001 0" rpy="0 0 0"/>
-      <geometry>
-        <box size="0.030 0.009 0.020"/>
-      </geometry>
-    </collision>
-    <inertial>
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
File: simplebot_description/urdf/simplebot.gazebo.macro.xacro (robot description, xacro)
@@ -104,5 +104,5 @@
       <pose>0 0 0 0 0 0</pose>
 <!--      <visualize>${laser_visual}</visualize>-->
-      <visualize>true</visualize>
+<!--      <visualize>true</visualize>-->
       <update_rate>5</update_rate>
       <ray>
@@ -137,5 +137,5 @@
       <pose>0 0 0 0 0 0</pose>
 <!--      <visualize>${laser_visual}</visualize>-->
-      <visualize>true</visualize>
+<!--      <visualize>true</visualize>-->
       <update_rate>5</update_rate>
       <ray>

File: simplebot_description/urdf/simplebot.urdf.xacro (robot description, xacro)
@@ -15,4 +15,5 @@
   <xacro:include filename="$(find simplebot_description)/urdf/VLP-16.urdf.xacro"/>
   <xacro:include filename="$(find simplebot_description)/urdf/astra.urdf.xacro" />
+  <xacro:include filename="$(find velodyne_description)/urdf/VLP-16.urdf.xacro"/>
   <xacro:include filename="$(find simplebot_description)/urdf/simplebot.gazebo.macro.xacro"/>
   <xacro:gazebo_macro color="$(arg color)" laser_visual="false" camera_visual="false" imu_visual="true"/>
@@ -205,21 +206,21 @@
     <origin xyz="-0.014 -0.05 0.222" rpy="0 0 0"/>
   </joint>
-<!--  <link name="lidar3d_plate_link">-->
-<!--    <visual>-->
-<!--      <origin xyz="0 0 0" rpy="0 0 0"/>-->
-<!--      <geometry>-->
-<!--        <box size="0.14 0.14 0.005"/>-->
-<!--      </geometry>-->
-<!--      <material name="grey"/>-->
-<!--    </visual>-->
-<!--  </link>-->
-<!--  <joint name="platform_support_leg1_link_to_lidar3d_plate_link" type="fixed">-->
-<!--    <parent link="platform_support_leg1_link"/>-->
-<!--    <child link="lidar3d_plate_link"/>-->
-<!--    <origin xyz="0.05 -0.05 0" rpy="0 0 0"/>-->
-<!--  </joint>-->
-<!--  <xacro:VLP-16 name="lidar3d" parent="lidar3d_plate_link" topic="/lidar3d/points">-->
-<!--    <origin xyz="0 0 0" rpy="0 0 0" />-->
-<!--  </xacro:VLP-16>-->
+  <!--  <link name="lidar3d_plate_link">-->
+  <!--    <visual>-->
+  <!--      <origin xyz="0 0 0" rpy="0 0 0"/>-->
+  <!--      <geometry>-->
+  <!--        <box size="0.14 0.14 0.005"/>-->
+  <!--      </geometry>-->
+  <!--      <material name="grey"/>-->
+  <!--    </visual>-->
+  <!--  </link>-->
+  <!--  <joint name="platform_support_leg1_link_to_lidar3d_plate_link" type="fixed">-->
+  <!--    <parent link="platform_support_leg1_link"/>-->
+  <!--    <child link="lidar3d_plate_link"/>-->
+  <!--    <origin xyz="0.05 -0.05 0" rpy="0 0 0"/>-->
+  <!--  </joint>-->
+  <!--  <xacro:VLP-16 name="lidar3d" parent="lidar3d_plate_link" topic="/lidar3d/points">-->
+  <!--    <origin xyz="0 0 0" rpy="0 0 0" />-->
+  <!--  </xacro:VLP-16>-->
   <link name="front_left_camera_support_link">
   </link>
@@ -232,29 +233,29 @@
     <origin xyz="0.02 0.07 0.015" rpy="0 0.0 0" />
   </xacro:sensor_astra>
-<!--  <link name="front_right_camera_support_link">-->
-<!--  </link>-->
-<!--  <joint name="platform_support_leg4_link_to_front_right_camera_support_link" type="fixed">-->
-<!--    <origin xyz="0.02 0 -0.05" rpy="0.01 -0.35 -0.22"/>-->
-<!--    <parent link="platform_support_leg4_link"/>-->
-<!--    <child link="front_right_camera_support_link"/>-->
-<!--  </joint>-->
-<!--  <xacro:sensor_astra prefix="front_right_camera" parent="front_right_camera_support_link">-->
-<!--    <origin xyz="0.02 0.07 0.015" rpy="0 0.0 0" />-->
-<!--  </xacro:sensor_astra>-->
-<!--  <link name="back_camera_support_link">-->
-<!--  </link>-->
-<!--  <joint name="platform_support_leg1_link_to_back_camera_support_link" type="fixed">-->
-<!--    <origin xyz="-0.02 -0.05 -0.10" rpy="0.01 -0.35 3.14"/>-->
-<!--    <parent link="platform_support_leg1_link"/>-->
-<!--    <child link="back_camera_support_link"/>-->
-<!--  </joint>-->
-<!--  <xacro:sensor_astra prefix="back_camera" parent="back_camera_support_link">-->
-<!--    <origin xyz="0.02 0.07 0.015" rpy="0 0.0 0" />-->
-<!--  </xacro:sensor_astra>-->
- <joint name="left_scan_joint" type="fixed">
+  <!--  <link name="front_right_camera_support_link">-->
+  <!--  </link>-->
+  <!--  <joint name="platform_support_leg4_link_to_front_right_camera_support_link" type="fixed">-->
+  <!--    <origin xyz="0.02 0 -0.05" rpy="0.01 -0.35 -0.22"/>-->
+  <!--    <parent link="platform_support_leg4_link"/>-->
+  <!--    <child link="front_right_camera_support_link"/>-->
+  <!--  </joint>-->
+  <!--  <xacro:sensor_astra prefix="front_right_camera" parent="front_right_camera_support_link">-->
+  <!--    <origin xyz="0.02 0.07 0.015" rpy="0 0.0 0" />-->
+  <!--  </xacro:sensor_astra>-->
+  <!--  <link name="back_camera_support_link">-->
+  <!--  </link>-->
+  <!--  <joint name="platform_support_leg1_link_to_back_camera_support_link" type="fixed">-->
+  <!--    <origin xyz="-0.02 -0.05 -0.10" rpy="0.01 -0.35 3.14"/>-->
+  <!--    <parent link="platform_support_leg1_link"/>-->
+  <!--    <child link="back_camera_support_link"/>-->
+  <!--  </joint>-->
+  <!--  <xacro:sensor_astra prefix="back_camera" parent="back_camera_support_link">-->
+  <!--    <origin xyz="0.02 0.07 0.015" rpy="0 0.0 0" />-->
+  <!--  </xacro:sensor_astra>-->
+  <joint name="left_scan_joint" type="fixed">
     <parent link="base_link"/>
     <child link="left_base_scan"/>
-<!--    <origin xyz="-0.064 0 0.122" rpy="0 0 0"/>-->
-   <origin xyz="0.037 0.1 0.122" rpy="0 0 0.78"/>
+    <!--    <origin xyz="-0.064 0 0.122" rpy="0 0 0"/>-->
+    <origin xyz="0.037 0.1 0.122" rpy="0 0 0.78"/>
   </joint>
   <link name="left_base_scan">
@@ -280,9 +281,9 @@
     </inertial>
   </link>
-   <joint name="right_scan_joint" type="fixed">
+  <joint name="right_scan_joint" type="fixed">
     <parent link="base_link"/>
     <child link="right_base_scan"/>
-<!--    <origin xyz="-0.064 0 0.122" rpy="0 0 0"/>-->
-   <origin xyz="0.037 -0.1 0.122" rpy="0 0 -0.78"/>
+    <!--    <origin xyz="-0.064 0 0.122" rpy="0 0 0"/>-->
+    <origin xyz="0.037 -0.1 0.122" rpy="0 0 -0.78"/>
   </joint>
   <link name="right_base_scan">
@@ -308,3 +309,7 @@
     </inertial>
   </link>
+  <!--  3d lidar-->
+  <xacro:VLP-16 name="lidar3d" parent="base_link" topic="/lidar3d/points">
+        <origin xyz="0 0 0.3" rpy="0 0 0" />
+  </xacro:VLP-16>
 </robot>
